File: hardware/cloud-substrate/cloud-substrate.sch (EAGLE design)
At the start: 113 parts

Commit message: Make pretty and HWB pin jumper point
Parts:
- added TP1: TEST-POINT2, SparkFun-Connectors:TEST-POINT2
- TP2: value TEST-POINT3X5 -> TEST-POINT2; device SparkFun-Connectors:TEST-POINT3X5 -> SparkFun-Connectors:TEST-POINT2
Connections:
- net GND: now also TP2.1
- net N$20: now also TP1.1; no longer TP2.1
Other:
- moved on the sheet: C1, C10, C11, C12, C2, C3, C4, C5, C6, C7, C8, C9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
